Commit message: maj urdf et gazebo

File: description/robot.urdf (robot description, URDF)
Before this commit: robot robot, 5 links, 4 joints
Links:
- link caster_wheel: geometry collision sphere radius=0.0325; visual sphere radius=0.0325
- link chassis: geometry collision cylinder length=0.005 radius=0.19; visual cylinder length=0.015 radius=0.19
- link left_wheel: geometry collision cylinder length=0.025 radius=0.0325; visual cylinder length=0.025 radius=0.0325
- link right_wheel: geometry collision cylinder length=0.025 radius=0.0325; visual cylinder length=0.025 radius=0.0325
Joints:
- joint caster_wheel_joint: origin xyz=0.24 0 0 rpy=0 0 0 -> xyz=0.25 0 0 rpy=0 0 0
- joint left_wheel_joint: origin xyz=0 0.175 0 rpy=-1.5707963267948966 0 0 -> xyz=-0.02 0.125 0 rpy=-1.5707963267948966 0 0
- joint right_wheel_joint: origin xyz=0 -0.175 0 rpy=1.5707963267948966 0 0 -> xyz=-0.02 -0.125 0 rpy=1.5707963267948966 0 0

File: description/robot_core.xacro (robot description, xacro)
@@ -25,18 +25,18 @@
     <link name="chassis">
         <visual>
-            <origin xyz="0.15 0 0.075" rpy="0 0 0"/>
+            <origin xyz="0.15 0 0.03" rpy="0 0 0"/>
             <geometry>
-                <box size="0.3 0.3 0.15"/>
+                <cylinder length="0.015" radius="0.19" />
             </geometry>
             <material name="white"/>
         </visual>
         <collision>
-            <origin xyz="0.15 0 0.075" rpy="0 0 0"/>
+            <origin xyz="0.15 0 0.03" rpy="0 0 0"/>
             <geometry>
-                <box size="0.3 0.3 0.15"/>
+                <cylinder length="0.005" radius="0.19" />
             </geometry>
         </collision>
         <xacro:inertial_box mass="0.5" x="0.3" y="0.3" z="0.15">
-            <origin xyz="0.15 0 0.075" rpy="0 0 0"/>
+            <origin xyz="0.15 0 0.03" rpy="0 0 0"/>
         </xacro:inertial_box>
     </link>
@@ -45,5 +45,5 @@
         <parent link="base_link"/>
         <child link="left_wheel"/>
-        <origin xyz="0 0.175 0" rpy="-${pi/2} 0 0"/>
+        <origin xyz="-0.02 0.125 0" rpy="-${pi/2} 0 0"/>
         <axis xyz="0 0 1"/>
     </joint>
@@ -51,5 +51,5 @@
         <visual>
             <geometry>
-                <cylinder length="0.04" radius="0.05" />
+                <cylinder length="0.025" radius="0.0325" />
             </geometry>
             <material name="blue"/>
@@ -57,8 +57,8 @@
         <collision>
             <geometry>
-                <cylinder length="0.04" radius="0.05" />
+                <cylinder length="0.025" radius="0.0325" />
             </geometry>
         </collision>
-        <xacro:inertial_cylinder mass="0.1" length="0.05" radius="0.05">
+        <xacro:inertial_cylinder mass="0.1" length="0.025" radius="0.0325">
             <origin xyz="0 0 0" rpy="0 0 0"/>
         </xacro:inertial_cylinder>
@@ -68,5 +68,5 @@
         <parent link="base_link"/>
         <child link="right_wheel"/>
-        <origin xyz="0 -0.175 0" rpy="${pi/2} 0 0"/>
+        <origin xyz="-0.02 -0.125 0" rpy="${pi/2} 0 0"/>
         <axis xyz="0 0 -1"/>
     </joint>
@@ -74,5 +74,5 @@
         <visual>
             <geometry>
-                <cylinder length="0.04" radius="0.05" />
+                <cylinder length="0.025" radius="0.0325" />
             </geometry>
             <material name="blue"/>
@@ -80,8 +80,8 @@
         <collision>
             <geometry>
-                <cylinder length="0.04" radius="0.05" />
+                <cylinder length="0.025" radius="0.0325" />
             </geometry>
         </collision>
-        <xacro:inertial_sphere mass="0.1" radius="0.05">
+        <xacro:inertial_sphere mass="0.1" radius="0.325">
             <origin xyz="0 0 0" rpy="0 0 0"/>
         </xacro:inertial_sphere>
@@ -91,10 +91,10 @@
         <parent link="chassis"/>
         <child link="caster_wheel"/>
-        <origin xyz="0.24 0 0" rpy="0 0 0"/>
+        <origin xyz="0.25 0 0" rpy="0 0 0"/>
     </joint>
     <link name="caster_wheel">
         <visual>
             <geometry>
-                <sphere radius="0.05" />
+                <sphere radius="0.0325" />
             </geometry>
             <material name="black"/>
@@ -102,5 +102,5 @@
         <collision>
             <geometry>
-                <sphere radius="0.05" />
+                <sphere radius="0.0325" />
             </geometry>
         </collision>
