Commit message: main

File: description/gazebo_control.xacro (robot description, xacro)
@@ -2,19 +2,31 @@
 <robot xmlns:xacro="http://www.ros.org/wiki/xacro">
     <gazebo>
-        <plugin name="diff_drive" filename="libgazebo_ros_diff_drive.so">
+        <plugin name="diff_drive_controller" filename="libgazebo_ros_diff_drive.so">
             <!--Wheel Information-->
-            <left_joint>left_wheel_joint</left_joint>
-            <right_joint>right_wheel_joint</right_joint>
-            <wheel_separation>0.35</wheel_separation>
-            <wheel_diameter>0.1</wheel_diameter>
+            <leftJoint>left_wheel_joint</leftJoint>
+            <rightJoint>right_wheel_joint</rightJoint>
+            <wheelSeparation>0.25</wheelSeparation>
+            <wheelDiameter>0.065</wheelDiameter>
             <!-- Limits -->
             <max_wheel_torque>200</max_wheel_torque>
             <max_wheel_acceleration>10.0</max_wheel_acceleration>
             <!-- Output -->
-            <odometry_frame>odom</odometry_frame>
-            <robot_base_frame>base_link</robot_base_frame>
-            <publish_odom>true</publish_odom>
-            <publish_odom_tf>true</publish_odom_tf>
-            <publish_wheel_tf>true</publish_wheel_tf>
+            <odometryFrame>odom</odometryFrame>
+            <robotBaseFrame>base_link</robotBaseFrame>
+            <publishOdom>true</publishOdom>
+            <publishOdomTF>true</publishOdomTF>
+            <publishWheelTF>true</publishWheelTF>
+            <!--Test with an other tutorial-->
+            <alwaysOn>true</alwaysOn>
+            <updateRate>10</updateRate>
+            <legacyMode>true</legacyMode>
+            <commandTopic>cmd_vel</commandTopic>
+            <odometryTopic>odom</odometryTopic>
+            <publishWheelJointState>true</publishWheelJointState>
+            <rosDebugLevel>na</rosDebugLevel>
+            <wheelAcceleration>10.0</wheelAcceleration>
+            <wheelTorque>200</wheelTorque>
+            <odometrySource>world</odometrySource>
+            <publishTf>1</publishTf>
         </plugin>
     </gazebo>

File: description/robot.urdf (robot description, URDF)
Before this commit: robot robot, 5 links, 4 joints
Links:
- added link laser_frame, mass 0.1; collision cylinder length=0.025 radius=0.0325; visual cylinder length=0.025 radius=0.0325
- link caster_wheel: mass None -> 0.1
- link chassis: mass 0.5 -> 4.0
Joints:
- added joint laser_joint: type fixed, parent chassis, child laser_frame, origin xyz=0.20 0 0.045 rpy=0 0 0

File: description/robot_core.xacro (robot description, xacro)
@@ -13,4 +13,7 @@
     <material name="black">
         <color rgba="0 0 0 1"/>
+    </material>
+    <material name="red">
+        <color rgba="1 0 0 1"/>
     </material>
 <!-- BASE LINK -->
@@ -37,7 +40,7 @@
             </geometry>
         </collision>
-        <xacro:inertial_box mass="0.5" x="0.3" y="0.3" z="0.15">
+        <xacro:inertial_cylinder mass="4.0" length="0.015" radius="0.19">
             <origin xyz="0.15 0 0.03" rpy="0 0 0"/>
-        </xacro:inertial_box>
+        </xacro:inertial_cylinder>
     </link>
     <gazebo reference="chassis">
@@ -113,8 +116,14 @@
                 <sphere radius="0.0325" />
             </geometry>
+            <material name="black"/>
         </collision>
+        <xacro:inertial_sphere mass="0.1" radius="0.0325">
+            <origin xyz="0 0 0" rpy="0 0 0"/>
+        </xacro:inertial_sphere>
     </link>
     <gazebo reference="caster_wheel">
         <material>Gazebo/Black</material>
+        <mu1 value="0"/>
+        <mu2 value="0"/>
     </gazebo>
 </robot>
