Commit message: main

File: description/lidar.xacro (robot description, xacro)
@@ -40,5 +40,5 @@
                     <min>0.3</min>
                     <max>12</max>
-                    <resolution>0.001</resolution>
+                    <resolution>0.01</resolution>
                 </range>
             </ray>

File: description/robot.urdf (robot description, URDF)
Before this commit: robot robot, 6 links, 5 joints
Links:
- added link base_footprint
Joints:
- added joint base_footprint_joint: type fixed, parent base_link, child base_footprint, origin xyz=0 0 0 rpy=0 0 0

File: description/robot_core.xacro (robot description, xacro)
@@ -19,4 +19,12 @@
 <!-- BASE LINK -->
     <link name="base_link">
+    </link>
+<!--BASE_FOOTPRINT LINK-->
+    <joint name="base_footprint_joint" type="fixed">
+        <parent link="base_link"/>
+        <child link="base_footprint"/>
+        <origin xyz="0 0 0" rpy="0 0 0"/>
+    </joint>
+    <link name="base_footprint">
     </link>
 <!-- CHASSIS LINK -->
